Commit message: add realsense to sim env

File: urdf/d435_camera.urdf.xacro (robot description, xacro)
@@ -2,11 +2,12 @@
 <robot name="realsense2_camera" xmlns:xacro="http://ros.org/wiki/xacro">
   <xacro:arg name="parent_link" default="world"/>
-  <xacro:arg name="use_nominal_extrinsics" default="false"/>
-  <xacro:arg name="add_plug" default="false" />
-  <xacro:arg name="use_mesh" default="true" />
   <xacro:include filename="$(find realsense2_description)/urdf/_d435.urdf.xacro" />
-  <link name="$(arg parent_link)"/>
-  <xacro:sensor_d435 parent="$(arg parent_link)" use_nominal_extrinsics="$(arg use_nominal_extrinsics)" add_plug="$(arg add_plug)" use_mesh="$(arg use_mesh)">
-    <origin xyz="0 0 0" rpy="0 0 0"/>
+  <link name="camera_base_link" />
+  <xacro:sensor_d435 name="camera" topics_ns="camera" parent="camera_base_link" publish_pointcloud="true">
+    <!-- <origin xyz="0 0.7 2" rpy="0 1.570796 1.570796" /> -->
+    <origin xyz="0 0 0" rpy="0 0 0" />
   </xacro:sensor_d435>
+  <gazebo>
+    <static>true</static>
+  </gazebo>
 </robot>

Commit message: add graspnet

File: urdf/d435_camera.urdf.xacro (robot description, xacro)
@@ -1,9 +1,7 @@
 <?xml version="1.0"?>
 <robot name="realsense2_camera" xmlns:xacro="http://ros.org/wiki/xacro">
-  <xacro:arg name="parent_link" default="world"/>
   <xacro:include filename="$(find realsense2_description)/urdf/_d435.urdf.xacro" />
   <link name="camera_base_link" />
-  <xacro:sensor_d435 name="camera" topics_ns="camera" parent="camera_base_link" publish_pointcloud="true">
-    <!-- <origin xyz="0 0.7 2" rpy="0 1.570796 1.570796" /> -->
+  <xacro:sensor_d435 name="camera" topics_ns="camera" parent="camera_base_link" publish_pointcloud="true" use_nominal_extrinsics="true">
     <origin xyz="0 0 0" rpy="0 0 0" />
   </xacro:sensor_d435>
